File: hardware/kicad/make_music.kicad_pcb (KiCad board)
At the start: 2 copper layers, 330 x 120 mm, 2 parts, among them J1 LEFT / Pico 1-20, J2 RIGHT / Pico 21-40

Commit message: Place carrier components and define module cable assembly
Parts:
- added C1: 100n, MakeMusicCarrier:KEMET_C0603_1608_LevelB, F.Cu at (96.5, 95.0)
- added C10: 100n, MakeMusicCarrier:KEMET_C0603_1608_LevelB, F.Cu at (50.5, 95.0)
- added C11: 100n, MakeMusicCarrier:KEMET_C0603_1608_LevelB, F.Cu at (87.5, 69.0)
- added C12: 100n, MakeMusicCarrier:KEMET_C0603_1608_LevelB, F.Cu at (125.5, 69.0)
- added C2: 100n, MakeMusicCarrier:KEMET_C0603_1608_LevelB, F.Cu at (130.5, 95.0)
- added C3: 100n, MakeMusicCarrier:KEMET_C0603_1608_LevelB, F.Cu at (164.5, 95.0)
- added C4: 100n, MakeMusicCarrier:KEMET_C0603_1608_LevelB, F.Cu at (198.5, 95.0)
- added C5: 100n, MakeMusicCarrier:KEMET_C0603_1608_LevelB, F.Cu at (232.5, 95.0)
- added C6: 100n, MakeMusicCarrier:KEMET_C0603_1608_LevelB, F.Cu at (266.5, 95.0)
- added C7: 100n, MakeMusicCarrier:KEMET_C0603_1608_LevelB, F.Cu at (300.5, 95.0)
- added C8: 100n, MakeMusicCarrier:KEMET_C0603_1608_LevelB, F.Cu at (334.5, 95.0)
- added C9: 100n, MakeMusicCarrier:KEMET_C0603_1608_LevelB, F.Cu at (50.5, 55.0)
- added D1: SS14-E3/61T, MakeMusicCarrier:Vishay_SS14_SMA_K1_A2, F.Cu at (236.0, 75.0)
- added H1: JST PH battery, Connector_JST:JST_PH_B2B-PH-K_1x02_P2.00mm_Vertical, B.Cu at (249.0, 40.0)
- added J10: C5 / GP26, MakeMusicCarrier:Harwin_M20-9990346_1x3_P2.54mm, F.Cu at (325.5, 95.0)
- added J11: Semitone up / GP27, MakeMusicCarrier:Harwin_M20-9990346_1x3_P2.54mm, F.Cu at (41.5, 55.0)
- added J12: Octave up / GP28, MakeMusicCarrier:Harwin_M20-9990346_1x3_P2.54mm, F.Cu at (41.5, 95.0)
- added J13: Buzzer 1 / PWM / GP13, MakeMusicCarrier:Harwin_M20-9990346_1x3_P2.54mm, F.Cu at (78.5, 69.0)
- added J14: Buzzer 2 / PWM / GP12, MakeMusicCarrier:Harwin_M20-9990346_1x3_P2.54mm, F.Cu at (116.5, 69.0)
- added J15: GPIO / Harwin 16-way, MakeMusicCarrier:Harwin_M20-9991646_1x16_P2.54mm, F.Cu at (70.0, 32.0)
- added J3: C4 / GP16, MakeMusicCarrier:Harwin_M20-9990346_1x3_P2.54mm, F.Cu at (87.5, 95.0)
- added J4: D4 / GP17, MakeMusicCarrier:Harwin_M20-9990346_1x3_P2.54mm, F.Cu at (121.5, 95.0)
- added J5: E4 / GP18, MakeMusicCarrier:Harwin_M20-9990346_1x3_P2.54mm, F.Cu at (155.5, 95.0)
- added J6: F4 / GP19, MakeMusicCarrier:Harwin_M20-9990346_1x3_P2.54mm, F.Cu at (189.5, 95.0)
- added J7: G4 / GP20, MakeMusicCarrier:Harwin_M20-9990346_1x3_P2.54mm, F.Cu at (223.5, 95.0)
- added J8: A4 / GP21, MakeMusicCarrier:Harwin_M20-9990346_1x3_P2.54mm, F.Cu at (257.5, 95.0)
- added J9: B4 / GP22, MakeMusicCarrier:Harwin_M20-9990346_1x3_P2.54mm, F.Cu at (291.5, 95.0)
- added MH1: MountingHole_3.2mm_M3, MountingHole_3.2mm_M3, F.Cu at (26.0, 26.0)
- added MH2: MountingHole_3.2mm_M3, MountingHole_3.2mm_M3, F.Cu at (344.0, 26.0)
- added MH3: MountingHole_3.2mm_M3, MountingHole_3.2mm_M3, F.Cu at (26.0, 134.0)
- added MH4: MountingHole_3.2mm_M3, MountingHole_3.2mm_M3, F.Cu at (344.0, 134.0)
- added MH5: MountingHole_3.2mm_M3, MountingHole_3.2mm_M3, F.Cu at (170.0, 37.0)
- added MH6: MountingHole_3.2mm_M3, MountingHole_3.2mm_M3, F.Cu at (230.0, 37.0)
- added MH7: MountingHole_3.2mm_M3, MountingHole_3.2mm_M3, F.Cu at (170.0, 63.0)
- added MH8: MountingHole_3.2mm_M3, MountingHole_3.2mm_M3, F.Cu at (230.0, 63.0)
- added R1: 10k, Resistor_SMD:R_0603_1608Metric, F.Cu at (79.0, 63.0)
- added R2: 10k, Resistor_SMD:R_0603_1608Metric, F.Cu at (117.0, 63.0)
- added S1: MN12SS1W03, MakeMusicCarrier:NKK_MN12SS1W03_TerminalPattern_Candidate, F.Cu at (270.0, 75.0)
Other:
- board text added: "1:S 2:3V3 3:G"
- board text added: "330 x 120; module body outlines are references; separate mounting fixture required"
- board text added: "BATTERY OFF"
- board text added: "EXPANSION 3.3V ONLY"
- board text added: "MAKE MUSIC - CARRIER P1"
- board text added: "OCTAVE"
- board text added: "OCTAVE +"
- board text added: "ON"
- board text added: "P1 CARRIER LAYOUT REVIEW - PHYSICAL FIT PENDING"
- board text added: "PICO - REMOVE POWER TO UNPLUG"
- board text added: "POWER CIRCUIT"
- board text added: "PROTOTYPE / FIT VALIDATION REQUIRED"
- board text added: "REMOVABLE PICO"
- board text added: "SEMITONE"
- board text added: "SEMITONE +"
- board text added: "ST0238 1"
- board text added: "ST0238 2"
- board text added: "TOUCH A4"
- board text added: "TOUCH B4"
- board text added: "TOUCH C4"
- board text added: "TOUCH C5"
- board text added: "TOUCH D4"
- board text added: "TOUCH E4"
- board text added: "TOUCH F4"
- board text added: "TOUCH G4"
- board text added: "UNDERSIDE INSULATING CASSETTE"
- board text removed: "330 x 120 mm proposed; paper fit and remaining parts pending"
- board text removed: "Body rectangles are reference drawings, not component footprints or mounting holes."
- board text removed: "GPIO HEADER - TBD"
- board text removed: "OCTAVE+"
- board text removed: "PICO USB END"
- board text removed: "PLACEMENT DRAFT - UNROUTED - NOT FOR FABRICATION"
- board text removed: "POWER PARTS - TBD"
- board text removed: "SEMITONE+"
- board text removed: "ST0238"
- board text removed: "UNDERSIDE BATTERY - MOUNT TBD"

Commit message: Route protected carrier and integrate module fixture mounts
Parts:
- removed D1: SS14-E3/61T, MakeMusicCarrier:Vishay_SS14_SMA_K1_A2
- added C13: 4u7 / 25V, Capacitor_SMD:C_0805_2012Metric, F.Cu at (238.8, 71.5)
- added C14: 4u7 / 25V, Capacitor_SMD:C_0805_2012Metric, F.Cu at (241.2, 80.5)
- added C15: 10n / 50V, Capacitor_SMD:C_0603_1608Metric, F.Cu at (247.0, 78.0)
- added C16: 4u7 / 25V, Capacitor_SMD:C_0805_2012Metric, F.Cu at (239.0, 87.0)
- added D2: SS14-E3/61T, MakeMusicCarrier:Vishay_SS14_SMA_K1_A2, F.Cu at (246.0, 83.5)
- added D3: SMAJ5.0CA, MakeMusicPower:Littelfuse_SMAJ5-0CA_DO-214AC, F.Cu at (248.0, 71.5)
- added F1: 1.25A T, MakeMusicPower:Schurter_UMT-H_3403-0275-23, F.Cu at (250.0, 50.0)
- added MH10: MountingHole_3.2mm_M3, MountingHole_3.2mm_M3, F.Cu at (65.0, 103.0)
- added MH11: MountingHole_3.2mm_M3, MountingHole_3.2mm_M3, F.Cu at (70.0, 134.0)
- added MH12: MountingHole_3.2mm_M3, MountingHole_3.2mm_M3, F.Cu at (175.0, 134.0)
- added MH13: MountingHole_3.2mm_M3, MountingHole_3.2mm_M3, F.Cu at (277.0, 134.0)
- added MH14: MountingHole_3.2mm_M3, MountingHole_3.2mm_M3, F.Cu at (311.0, 134.0)
- added MH15: MountingHole_3.2mm_M3, MountingHole_3.2mm_M3, F.Cu at (175.0, 93.0)
- added MH16: MountingHole_3.2mm_M3, MountingHole_3.2mm_M3, F.Cu at (209.0, 93.0)
- added MH17: MountingHole_3.2mm_M3, MountingHole_3.2mm_M3, F.Cu at (311.0, 93.0)
- added MH9: MountingHole_3.2mm_M3, MountingHole_3.2mm_M3, F.Cu at (28.0, 94.0)
- added R3: 649k, Resistor_SMD:R_0603_1608Metric, F.Cu at (235.0, 73.0)
- added R4: 332k, Resistor_SMD:R_0603_1608Metric, F.Cu at (235.0, 75.0)
- added R5: 1.05M, Resistor_SMD:R_0603_1608Metric, F.Cu at (235.0, 78.5)
- added R6: 332k, Resistor_SMD:R_0603_1608Metric, F.Cu at (235.0, 80.5)
- added R7: 3.32k, Resistor_SMD:R_0603_1608Metric, F.Cu at (244.0, 74.3)
- added R8: 100, Resistor_SMD:R_0603_1608Metric, F.Cu at (244.0, 78.0)
- added TP1: USB VBUS only, TestPoint:TestPoint_Pad_D2.0mm, F.Cu at (157.0, 23.0)
- added U2: TPS259474LRPWR, MakeMusicPower:TI_RPW0010A_TPS259474_2x2mm, F.Cu at (240.0, 76.0)
Connections:
- H1 pad 1: /BAT_PROT_PLUS -> /Battery protection/BAT_PROT_PLUS
- S1 pad 2: /BAT_PROT_PLUS -> /Battery protection/BAT_FUSED_PLUS
- S1 pad 3: /BAT_SW_PLUS -> /Battery protection/BAT_SW_PLUS
Routing:
- net /GND: track 0.00 -> 639.2 mm, vias 0 -> 24
- net /3V3_OUT: track 0.00 -> 576.1 mm, vias 0 -> 1
- net /GP26: track 0.00 -> 210.2 mm, vias 0 -> 1
- net /GP22: track 0.00 -> 184.2 mm, vias 0 -> 1
- net /GP21: track 0.00 -> 155.4 mm, vias 0 -> 1
- net /GP28: track 0.00 -> 135.0 mm
- net /VSYS: track 0.00 -> 131.5 mm, vias 0 -> 1
- net /GP27: track 0.00 -> 125.7 mm, vias 0 -> 1
- net /GP20: track 0.00 -> 90.4 mm, vias 0 -> 1
- net /GP16: track 0.00 -> 79.9 mm
- net /Battery protection/BAT_SW_PLUS: track 0.00 -> 68.4 mm
- net /GP15: track 0.00 -> 67.0 mm
- net /GP14: track 0.00 -> 67.0 mm
- net /GP13: track 0.00 -> 66.8 mm
- net /GP1: track 0.00 -> 65.5 mm
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- added copper zone on B.Cu, net /GND
- added copper zone on F.Cu, net /GND
Other:
- board text added: "1 +"
- board text added: "2 GND"
- board text added: "3V3"
- board text added: "GND"
- board text added: "GP0"
- board text added: "GP1"
- board text added: "GP10"
- board text added: "GP11"
- board text added: "GP14"
- board text added: "GP15"
- board text added: "GP2"
- board text added: "GP3"
- board text added: "GP4"
- board text added: "GP5"
- board text added: "GP6"
- board text added: "GP7"
- board text added: "GP8"
- board text added: "GP9"
- board text added: "PROTECTED 1S / EXTERNAL CHARGE"
