File: hardware/kicad/make_music.kicad_sch (KiCad schematic)
At the start: 33 parts, among them J1 LEFT / Pico 1-20, J10 C5 / GP26, J11 Semitone up / GP27, J12 Octave up / GP28, J13 Buzzer 1 / PWM / GP13, J14 Buzzer 2 / PWM / GP12, J15 GPIO / Harwin 16-way, J2 RIGHT / Pico 21-40, J3 C4 / GP16, J4 D4 / GP17, J5 E4 / GP18, J6 F4 / GP19, J7 G4 / GP20, J8 A4 / GP21, J9 B4 / GP22

Commit message: Integrate fused TPS259474L battery protection into native schematic
Parts:
- removed D1: SS14-E3/61T, MakeMusicCarrier:Vishay_SS14_SMA_K1_A2, symbol MakeMusic:SS14_K1_A2
- removed H1: JST PH battery, Connector_JST:JST_PH_B2B-PH-K_1x02_P2.00mm_Vertical, symbol MakeMusic:JST_PH_Battery_Harness
- removed S1: MN12SS1W03, MakeMusicCarrier:NKK_MN12SS1W03_TerminalPattern_Candidate, symbol MakeMusic:NKK_MN12_Common2
- TP1: footprint (none) -> TestPoint:TestPoint_Pad_D2.0mm; now left out of the parts list
Connections:
- no-connect marks 4 -> 3
Other:
- added sheet Battery protection (battery_power.kicad_sch)
- note added: "ERC checks carrier wiring only. Cell PCM, module electronics and assembled fault/load/fit behavior remain unverified. See power sheet."
- note added: "External charging only; cell/holder fit still pending."
- note added: "F1 + U2 replace the old carrier series D1."
- note added: "FUSED BATTERY POWER - SHEET 2"
- note added: "H1 JST harness: circuit1 protected positive, circuit2 GND."
- note added: "Selected Pico H SC0917: original RP2040, fitted male headers. Socket pitch2.54mm / rows17.78mm; fit trial pending."
- note added: "Sources: Raspberry Pi original Pico datasheet, Figure 2 pin allocation; see ../reviews/schematic.md."
- note added: "Stop playing before source changes; reboot may occur."
- note added: "Switch OFF isolates battery; USB may still power Pico."
- note removed: "Branch fuse/current limit and PCM cutoff remain TBD."
- note removed: "Cell/L1 charger are review targets, not approved parts."
- note removed: "ERC checks carrier wiring only. Cell PCM, branch fault limits, module electronics and load/fit remain unverified."
- note removed: "H1 JST PH: circuit 1=BAT_PROT_PLUS, circuit 2=GND."
- note removed: "K / band"
- note removed: "No carrier VBUS bridge; no onboard charger."
- note removed: "OFF:1 NC"
- note removed: "REV1 EXTERNAL-CHARGE BATTERY POWER"
- note removed: "Remove cell for external charging; see power handoff."
- note removed: "S1 OFF isolates battery; USB can still power Pico."
- note removed: "Sources: Raspberry Pi Pico/Pico 2 datasheets, Figure 2 pin allocation; see ../reviews/schematic.md."
- note removed: "Two 1x20 female sockets: 2.54 mm pitch, 17.78 mm row spacing. Carrier contacts are passive."
- note removed: "USB -> Pico onboard diode -> VSYS (inside Pico)."
- note removed: "Wired 1101 cassette approved; protected-cell fit pending."
- company: Review only - parts and power unresolved -> Prototype review - fit and bench validation pending

Commit message: Add buzzer bulk bypass and native socket purchasing fields
Parts:
- added C17, C18: 10u / 10V, Capacitor_SMD:C_0805_2012Metric, symbol Device:C
- J1, J2: MPN (none) -> SSQ-120-01-G-S
Connections:
- net 3V3_OUT: now also C17.1, C18.1
- net GND: now also C17.2, C18.2
Other:
- note added: "C17/J13: 10uF; retain C11 100nF. Place at buzzer header."
- note added: "C18/J14: 10uF; retain C12 100nF. Place at buzzer header."
